File: 8884bt Remote Control Receiver/board/Brickster 8884bt Receiver.brd (EAGLE design)
At the start: 28.8 x 28.8 mm, 22 parts, among them IC2 IC_RT9164A, J1 AVR_SPI_PRG_6NS, J2 CON_PF, J3 CON_PF, J4 CON_PF, U1 IC_ATTINY_X4A, U2 IC_TB6612FNG

Commit message: Fix D2/Bluetooth intersection
Parts:
- moved D2 1.57 mm to (2.74, 4.70), turned to 180 degrees
Routing:
- net VIN: track 62.9 -> 64.2 mm
- net N$1: track 17.8 -> 16.5 mm
Changed lines of the file:
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@@
 <?xml version="1.0" encoding="utf-8"?>
 <!DOCTYPE eagle SYSTEM "eagle.dtd">
-<eagle version="6.4">
+<eagle version="6.5.0">
 <drawing>
 <settings>
@@
 <attribute name="NAME" x="17.7198" y="1.8288" size="0.6096" layer="25" rot="R90" align="bottom-center"/>
 </element>
-<element name="D2" library="brickster" package="SOD80" value="D" x="4.2926" y="4.953" smashed="yes" rot="MR270">
-<attribute name="NAME" x="3.2926" y="4.953" size="0.6096" layer="26" rot="MR270" align="bottom-center"/>
+<element name="D2" library="brickster" package="SOD80" value="D" x="2.7432" y="4.699" smashed="yes" rot="MR180">
+<attribute name="NAME" x="2.7432" y="3.699" size="0.6096" layer="26" rot="MR180" align="bottom-center"/>
 </element>
 <element name="J2" library="brickster" package="CON_PF" value="CON_PF" x="14.3764" y="0.9398"/>
@@
 <wire x1="20.5042" y1="11.8412" x2="19.3086" y2="11.8412" width="0.1524" layer="1"/>
 <wire x1="19.3086" y1="11.8412" x2="19.3086" y2="11.4534" width="0.1524" layer="1"/>
-<wire x1="4.2926" y1="3.403" x2="4.2926" y2="2.2606" width="0.1524" layer="16"/>
+<wire x1="4.2932" y1="4.699" x2="4.2926" y2="2.2606" width="0.1524" layer="16"/>
 <wire x1="27.054" y1="8.7884" x2="27.054" y2="9.8298" width="0.1524" layer="1"/>
 </signal>
@@
 <contactref element="D2" pad="1"/>
 <wire x1="1.6764" y1="19.304" x2="0.508" y2="19.304" width="0.1524" layer="16"/>
-<wire x1="0.508" y1="19.304" x2="0.508" y2="6.503" width="0.1524" layer="16"/>
-<wire x1="0.508" y1="6.503" x2="4.2926" y2="6.503" width="0.1524" layer="16"/>
+<wire x1="0.508" y1="19.304" x2="0.508" y2="4.699" width="0.1524" layer="16"/>
+<wire x1="0.508" y1="4.699" x2="1.1932" y2="4.699" width="0.1524" layer="16"/>
 </signal>
 </signals>
